Commit message: Add goal control logic with exclusive region assignment.
Split long goals into outer side prisms in URDF/YAML and teach goal_reader to publish per-side control from min/max Y blocks without double-counting overlapping regions.

Co-authored-by: Cursor <cursoragent@cursor.com>

File: 03_ROS/ghost_localization/maps/pushBackField.urdf (robot description, URDF)
Before this commit: robot push_back_field, 1 links, 0 joints
Links:
- link map: geometry collision box size=0.481 0.15 0.15; collision box size=0.481 0.15 0.15
